File: allZones/allZones.kicad_sch (KiCad schematic)
At the start: 273 parts

Commit message: Added Missing #OE Connection
Connections:
- net at U?.23 (#OE): now also U?.23 (#OE), U?.23 (#OE), U?.23 (#OE), U?.23 (#OE), U?.23 (#OE), U?.23 (#OE), U?.23 (#OE), U?.23 (#OE), U?.23 (#OE), U?.23 (#OE), U?.23 (#OE), U?.23 (#OE), U?.23 (#OE), U?.23 (#OE), U?.23 (#OE)

Commit message: Fixed Again
Parts:
- removed M? (x192): Motor_Servo, symbol Motor:Motor_Servo
- removed U? (x12): PCA9685, symbol PWM:PCA9685
- added M? (x128): Motor_Servo, symbol Motor:Motor_Servo
- added U? (x8): PCA9685, symbol PWM:PCA9685
- added XA? (x11): Arduino_Uno_Shield, Arduino_Library:Arduino_Uno_Shield, symbol arduino:Arduino_Uno_Shield
Connections:
- net +5V: now also M?.2 (+), M?.2 (+), M?.2 (+), M?.2 (+), M?.2 (+), M?.2 (+), M?.2 (+), M?.2 (+), M?.2 (+), M?.2 (+), M?.2 (+), M?.2 (+), M?.2 (+), M?.2 (+), M?.2 (+), M?.2 (+), M?.2 (+), M?.2 (+), M?.2 (+), M?.2 (+), M?.2 (+), M?.2 (+), M?.2 (+), M?.2 (+), M?.2 (+), M?.2 (+), M?.2 (+), M?.2 (+), M?.2 (+), M?.2 (+), M?.2 (+), M?.2 (+), M?.2 (+), M?.2 (+), M?.2 (+), M?.2 (+), M?.2 (+), M?.2 (+), M?.2 (+), M?.2 (+), M?.2 (+), M?.2 (+), M?.2 (+), M?.2 (+), M?.2 (+), M?.2 (+), M?.2 (+), M?.2 (+), M?.2 (+), M?.2 (+), M?.2 (+), M?.2 (+), M?.2 (+), M?.2 (+), M?.2 (+), M?.2 (+), M?.2 (+), M?.2 (+), M?.2 (+), M?.2 (+), M?.2 (+), M?.2 (+), M?.2 (+), M?.2 (+), M?.2 (+), M?.2 (+), M?.2 (+), M?.2 (+), M?.2 (+), M?.2 (+), M?.2 (+), M?.2 (+), M?.2 (+), M?.2 (+), M?.2 (+), M?.2 (+), M?.2 (+), M?.2 (+), M?.2 (+), M?.2 (+), M?.2 (+), M?.2 (+), M?.2 (+), M?.2 (+), M?.2 (+), M?.2 (+), M?.2 (+), M?.2 (+), M?.2 (+), M?.2 (+), M?.2 (+), M?.2 (+), M?.2 (+), M?.2 (+), M?.2 (+), M?.2 (+), M?.2 (+), M?.2 (+), M?.2 (+), M?.2 (+), M?.2 (+), M?.2 (+), M?.2 (+), M?.2 (+), M?.2 (+), M?.2 (+), M?.2 (+), M?.2 (+), M?.2 (+), M?.2 (+), M?.2 (+), M?.2 (+), M?.2 (+), M?.2 (+), M?.2 (+), M?.2 (+), M?.2 (+), M?.2 (+), M?.2 (+), M?.2 (+), M?.2 (+), M?.2 (+), M?.2 (+), M?.2 (+), M?.2 (+), M?.2 (+), M?.2 (+), M?.2 (+), U?.28 (VDD), U?.28 (VDD), U?.28 (VDD), U?.28 (VDD), U?.28 (VDD), U?.28 (VDD), U?.28 (VDD), U?.28 (VDD)
- net +9V: now also XA?.VIN, XA?.VIN, XA?.VIN, XA?.VIN, XA?.VIN, XA?.VIN, XA?.VIN, XA?.VIN, XA?.VIN, XA?.VIN, XA?.VIN
- net GND: now also M?.3 (-), M?.3 (-), M?.3 (-), M?.3 (-), M?.3 (-), M?.3 (-), M?.3 (-), M?.3 (-), M?.3 (-), M?.3 (-), M?.3 (-), M?.3 (-), M?.3 (-), M?.3 (-), M?.3 (-), M?.3 (-), M?.3 (-), M?.3 (-), M?.3 (-), M?.3 (-), M?.3 (-), M?.3 (-), M?.3 (-), M?.3 (-), M?.3 (-), M?.3 (-), M?.3 (-), M?.3 (-), M?.3 (-), M?.3 (-), M?.3 (-), M?.3 (-), M?.3 (-), M?.3 (-), M?.3 (-), M?.3 (-), M?.3 (-), M?.3 (-), M?.3 (-), M?.3 (-), M?.3 (-), M?.3 (-), M?.3 (-), M?.3 (-), M?.3 (-), M?.3 (-), M?.3 (-), M?.3 (-), M?.3 (-), M?.3 (-), M?.3 (-), M?.3 (-), M?.3 (-), M?.3 (-), M?.3 (-), M?.3 (-), M?.3 (-), M?.3 (-), M?.3 (-), M?.3 (-), M?.3 (-), M?.3 (-), M?.3 (-), M?.3 (-), M?.3 (-), M?.3 (-), M?.3 (-), M?.3 (-), M?.3 (-), M?.3 (-), M?.3 (-), M?.3 (-), M?.3 (-), M?.3 (-), M?.3 (-), M?.3 (-), M?.3 (-), M?.3 (-), M?.3 (-), M?.3 (-), M?.3 (-), M?.3 (-), M?.3 (-), M?.3 (-), M?.3 (-), M?.3 (-), M?.3 (-), M?.3 (-), M?.3 (-), M?.3 (-), M?.3 (-), M?.3 (-), M?.3 (-), M?.3 (-), M?.3 (-), M?.3 (-), M?.3 (-), M?.3 (-), M?.3 (-), M?.3 (-), M?.3 (-), M?.3 (-), M?.3 (-), M?.3 (-), M?.3 (-), M?.3 (-), M?.3 (-), M?.3 (-), M?.3 (-), M?.3 (-), M?.3 (-), M?.3 (-), M?.3 (-), M?.3 (-), M?.3 (-), M?.3 (-), M?.3 (-), M?.3 (-), M?.3 (-), M?.3 (-), M?.3 (-), M?.3 (-), M?.3 (-), M?.3 (-), M?.3 (-), M?.3 (-), M?.3 (-), M?.3 (-), XA?.GND1 (GND), XA?.GND1 (GND), XA?.GND1 (GND), XA?.GND1 (GND), XA?.GND1 (GND), XA?.GND1 (GND), XA?.GND1 (GND), XA?.GND1 (GND), XA?.GND1 (GND), XA?.GND1 (GND), XA?.GND1 (GND)
- net at U?.26 (SCL), U?.26 (SCL), U?.26 (SCL)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: now also U?.26 (SCL), U?.26 (SCL), U?.26 (SCL), U?.26 (SCL), U?.26 (SCL), U?.26 (SCL), U?.26 (SCL), U?.26 (SCL), XA?.SCL, XA?.SCL, XA?.SCL, XA?.SCL, XA?.SCL, XA?.SCL, XA?.SCL, XA?.SCL, XA?.SCL, XA?.SCL, XA?.SCL
- net at U?.27 (SDA), U?.27 (SDA), U?.27 (SDA)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: now also U?.27 (SDA), U?.27 (SDA), U?.27 (SDA), U?.27 (SDA), U?.27 (SDA), U?.27 (SDA), U?.27 (SDA), U?.27 (SDA), XA?.SDA, XA?.SDA, XA?.SDA, XA?.SDA, XA?.SDA, XA?.SDA, XA?.SDA, XA?.SDA, XA?.SDA, XA?.SDA, XA?.SDA
- new net: M?.1 (PWM), U?.12 (PWM6) (x8)
- new net: M?.1 (PWM), U?.19 (PWM12) (x8)
- new net: M?.1 (PWM), U?.10 (PWM4) (x8)
- new net: M?.1 (PWM), U?.11 (PWM5) (x8)
- new net: M?.1 (PWM), U?.13 (PWM7) (x8)
- new net: M?.1 (PWM), U?.15 (PWM8) (x8)
- new net: M?.1 (PWM), U?.16 (PWM9) (x8)
- new net: M?.1 (PWM), U?.17 (PWM10) (x8)
- new net: M?.1 (PWM), U?.18 (PWM11) (x8)
- new net: M?.1 (PWM), U?.20 (PWM13) (x8)
- new net: M?.1 (PWM), U?.21 (PWM14) (x8)
- new net: M?.1 (PWM), U?.22 (PWM15) (x8)
- new net: U?.23 (#OE), U?.23 (#OE), U?.23 (#OE), U?.23 (#OE)
- new net: M?.1 (PWM), U?.6 (PWM0) (x8)
- new net: M?.1 (PWM), U?.7 (PWM1) (x8)
- new net: M?.1 (PWM), U?.8 (PWM2) (x8)
- new net: M?.1 (PWM), U?.9 (PWM3) (x8)
- now unconnected: U?.23 (#OE), U?.23 (#OE), U?.23 (#OE), U?.23 (#OE)
Other:
- moved on the sheet: M?, U?, XA?
